Commit message: updates
Signed-off-by: Kenji Brameld <kenjibrameld@gmail.com>

File: walk_bot/urdf/walk_bot.urdf (robot description, URDF)
Before this commit: robot walk_bot, 15 links, 14 joints
Links:
- link l_ankle1: mass 1.02 -> 0.001
- link l_ankle2: mass 1.02 -> 0.001
- link l_ankle3: mass 1.02 -> 0.001
- link l_hip1: mass 1.02 -> 0.001
- link l_hip2: mass 1.02 -> 0.001
- link l_hip3: mass 1.02 -> 0.001
- link l_sole: mass 1.02 -> 0.001
- link r_ankle1: mass 1.02 -> 0.001
- link r_ankle2: mass 1.02 -> 0.001
- link r_ankle3: mass 1.02 -> 0.001
- link r_hip1: mass 1.02 -> 0.001
- link r_hip2: mass 1.02 -> 0.001
- link r_hip3: mass 1.02 -> 0.001
- link r_sole: mass 1.02 -> 0.001
Joints:
- joint l_ankle_pitch: limit (none) -> lower=-3.14 upper=3.14 effort=1000.0 velocity=1000.0; type continuous -> revolute
- joint l_ankle_roll: limit (none) -> lower=-3.14 upper=3.14 effort=1000.0 velocity=1000.0; type continuous -> revolute
- joint l_hip_pitch: limit (none) -> lower=-3.14 upper=3.14 effort=1000.0 velocity=1000.0; type continuous -> revolute
- joint l_hip_roll: limit (none) -> lower=-3.14 upper=3.14 effort=1000.0 velocity=1000.0; type continuous -> revolute
- joint l_hip_yaw: limit (none) -> lower=-3.14 upper=3.14 effort=1000.0 velocity=1000.0; type continuous -> revolute
- joint l_leg_extension: limit lower=-0.4 upper=-0.2 effort=1000.0 velocity=1.0 -> lower=-0.4 upper=-0.2 effort=1000.0 velocity=1000.0
- joint r_ankle_pitch: limit (none) -> lower=-3.14 upper=3.14 effort=1000.0 velocity=1000.0; type continuous -> revolute
- joint r_ankle_roll: limit (none) -> lower=-3.14 upper=3.14 effort=1000.0 velocity=1000.0; type continuous -> revolute
- joint r_hip_pitch: limit (none) -> lower=-3.14 upper=3.14 effort=1000.0 velocity=1000.0; type continuous -> revolute
- joint r_hip_roll: limit (none) -> lower=-3.14 upper=3.14 effort=1000.0 velocity=1000.0; type continuous -> revolute
- joint r_hip_yaw: limit (none) -> lower=-3.14 upper=3.14 effort=1000.0 velocity=1000.0; type continuous -> revolute
- joint r_leg_extension: limit lower=-0.4 upper=-0.2 effort=1000.0 velocity=1.0 -> lower=-0.4 upper=-0.2 effort=1000.0 velocity=1000.0

Commit message: removee ankle to sole
Signed-off-by: Kenji Brameld <kenjibrameld@gmail.com>

File: walk_bot/urdf/walk_bot.urdf (robot description, URDF)
Before this commit: robot walk_bot, 15 links, 14 joints
Links:
- removed link l_ankle3
- removed link r_ankle3
Joints:
- removed joint l_sole_offset
- removed joint r_sole_offset
- joint l_ankle_pitch: child l_ankle3 -> l_sole
- joint r_ankle_pitch: child r_ankle3 -> r_sole

Commit message: ik working up to sole pose (no orientation yet)
Signed-off-by: Kenji Brameld <kenjibrameld@gmail.com>

File: walk_bot/urdf/walk_bot.urdf (robot description, URDF)
Before this commit: robot walk_bot, 13 links, 12 joints
Joints:
- joint l_hip_roll: origin xyz=0 0.1 0 rpy=0 0 0 -> xyz=0 0 0 rpy=0 0 0
- joint l_leg_extension: axis 0 0 1 -> 0 0 -1; limit lower=-0.4 upper=-0.2 effort=1000.0 velocity=1000.0 -> lower=0.2 upper=0.4 effort=1000.0 velocity=1000.0
- joint r_hip_roll: origin xyz=0 -0.1 0 rpy=0 0 0 -> xyz=0 0 0 rpy=0 0 0
- joint r_leg_extension: axis 0 0 1 -> 0 0 -1; limit lower=-0.4 upper=-0.2 effort=1000.0 velocity=1000.0 -> lower=0.2 upper=0.4 effort=1000.0 velocity=1000.0

Commit message: start getting ankle quaternion working
Signed-off-by: Kenji Brameld <kenjibrameld@gmail.com>

File: walk_bot/urdf/walk_bot.urdf (robot description, URDF)
Before this commit: robot walk_bot, 13 links, 12 joints
Links:
- removed link l_hip3
- removed link r_hip3
- added link l_ankle3, mass 0.001
- added link r_ankle3, mass 0.001
Joints:
- removed joint l_hip_yaw
- removed joint r_hip_yaw
- added joint l_ankle_yaw: type revolute, parent l_ankle1, child l_ankle2, axis 0 0 1, limit lower=-3.14 upper=3.14 effort=1000.0 velocity=1000.0
- added joint r_ankle_yaw: type revolute, parent r_ankle1, child r_ankle2, axis 0 0 1, limit lower=-3.14 upper=3.14 effort=1000.0 velocity=1000.0
- joint l_ankle_pitch: child l_sole -> l_ankle3
- joint l_ankle_roll: child l_ankle2 -> l_sole; parent l_ankle1 -> l_ankle3
- joint l_leg_extension: parent l_hip3 -> l_hip2
- joint r_ankle_pitch: child r_sole -> r_ankle3
- joint r_ankle_roll: child r_ankle2 -> r_sole; parent r_ankle1 -> r_ankle3
- joint r_leg_extension: parent r_hip3 -> r_hip2

Commit message: got ik working!
Signed-off-by: Kenji Brameld <kenjibrameld@gmail.com>

File: walk_bot/urdf/walk_bot.urdf (robot description, URDF)
Before this commit: robot walk_bot, 13 links, 12 joints
Joints:
- joint l_hip_pitch: child l_hip2 -> l_hip1; origin (none) -> xyz=0 0 0 rpy=0 0 0; parent l_hip1 -> base_link
- joint l_hip_roll: child l_hip1 -> l_hip2; origin xyz=0 0 0 rpy=0 0 0 -> (none); parent base_link -> l_hip1
- joint r_hip_pitch: child r_hip2 -> r_hip1; origin (none) -> xyz=0 0 0 rpy=0 0 0; parent r_hip1 -> base_link
- joint r_hip_roll: child r_hip1 -> r_hip2; origin xyz=0 0 0 rpy=0 0 0 -> (none); parent base_link -> r_hip1

Commit message: more sensible values in walk_bot.urdf
Signed-off-by: Kenji Brameld <kenjibrameld@gmail.com>

File: walk_bot/urdf/walk_bot.urdf (robot description, URDF)
Before this commit: robot walk_bot, 13 links, 12 joints
Links:
- link base_link: mass 1.02 -> 1.00
- link l_sole: mass 0.001 -> 0.3; geometry collision box size=0.15 0.05 0.02; visual box size=0.15 0.05 0.02
- link r_sole: mass 0.001 -> 0.3; geometry collision box size=0.15 0.05 0.02; visual box size=0.15 0.05 0.02
Joints:
- joint l_ankle_pitch: limit lower=-3.14 upper=3.14 effort=1000.0 velocity=1000.0 -> lower=-3.14 upper=3.14 effort=20.0 velocity=2.0
- joint l_ankle_roll: limit lower=-3.14 upper=3.14 effort=1000.0 velocity=1000.0 -> lower=-3.14 upper=3.14 effort=20.0 velocity=2.0
- joint l_ankle_yaw: limit lower=-3.14 upper=3.14 effort=1000.0 velocity=1000.0 -> lower=-3.14 upper=3.14 effort=20.0 velocity=2.0
- joint l_hip_pitch: limit lower=-3.14 upper=3.14 effort=1000.0 velocity=1000.0 -> lower=-3.14 upper=3.14 effort=20.0 velocity=2.0
- joint l_hip_roll: limit lower=-3.14 upper=3.14 effort=1000.0 velocity=1000.0 -> lower=-3.14 upper=3.14 effort=20.0 velocity=2.0
- joint l_leg_extension: limit lower=0.2 upper=0.4 effort=1000.0 velocity=1000.0 -> lower=0.2 upper=0.4 effort=20.0 velocity=2.0
- joint r_ankle_pitch: limit lower=-3.14 upper=3.14 effort=1000.0 velocity=1000.0 -> lower=-3.14 upper=3.14 effort=20.0 velocity=2.0
- joint r_ankle_roll: limit lower=-3.14 upper=3.14 effort=1000.0 velocity=1000.0 -> lower=-3.14 upper=3.14 effort=20.0 velocity=2.0
- joint r_ankle_yaw: limit lower=-3.14 upper=3.14 effort=1000.0 velocity=1000.0 -> lower=-3.14 upper=3.14 effort=20.0 velocity=2.0
- joint r_hip_pitch: limit lower=-3.14 upper=3.14 effort=1000.0 velocity=1000.0 -> lower=-3.14 upper=3.14 effort=20.0 velocity=2.0
- joint r_hip_roll: limit lower=-3.14 upper=3.14 effort=1000.0 velocity=1000.0 -> lower=-3.14 upper=3.14 effort=20.0 velocity=2.0
- joint r_leg_extension: limit lower=0.2 upper=0.4 effort=1000.0 velocity=1000.0 -> lower=0.2 upper=0.4 effort=20.0 velocity=2.0

Commit message: tuned joint pids
Signed-off-by: ijnek <kenjibrameld@gmail.com>

File: walk_bot/urdf/walk_bot.urdf (robot description, URDF)
Before this commit: robot walk_bot, 14 links, 13 joints
Joints:
- joint l_ankle_pitch: limit lower=-3.14 upper=3.14 effort=20.0 velocity=2.0 -> lower=-3.14 upper=3.14 effort=20.0 velocity=6.0
- joint l_ankle_roll: limit lower=-3.14 upper=3.14 effort=20.0 velocity=2.0 -> lower=-3.14 upper=3.14 effort=20.0 velocity=6.0
- joint l_ankle_yaw: limit lower=-3.14 upper=3.14 effort=20.0 velocity=2.0 -> lower=-3.14 upper=3.14 effort=20.0 velocity=6.0
- joint l_hip_pitch: limit lower=-3.14 upper=3.14 effort=20.0 velocity=2.0 -> lower=-3.14 upper=3.14 effort=20.0 velocity=6.0
- joint l_hip_roll: limit lower=-3.14 upper=3.14 effort=20.0 velocity=2.0 -> lower=-3.14 upper=3.14 effort=20.0 velocity=6.0
- joint r_ankle_pitch: limit lower=-3.14 upper=3.14 effort=20.0 velocity=2.0 -> lower=-3.14 upper=3.14 effort=20.0 velocity=6.0
- joint r_ankle_roll: limit lower=-3.14 upper=3.14 effort=20.0 velocity=2.0 -> lower=-3.14 upper=3.14 effort=20.0 velocity=6.0
- joint r_ankle_yaw: limit lower=-3.14 upper=3.14 effort=20.0 velocity=2.0 -> lower=-3.14 upper=3.14 effort=20.0 velocity=6.0
- joint r_hip_pitch: limit lower=-3.14 upper=3.14 effort=20.0 velocity=2.0 -> lower=-3.14 upper=3.14 effort=20.0 velocity=6.0
- joint r_hip_roll: limit lower=-3.14 upper=3.14 effort=20.0 velocity=2.0 -> lower=-3.14 upper=3.14 effort=20.0 velocity=6.0
